Commit message: amr description pkg

File: src/amr_description/urdf/amr.urdf.xacro (robot description, xacro)
@@ -1,13 +1,335 @@
-    <robot name="my_amr">
-        <link name="base_footprint"/>
-        <link name="base">
-        <inertial>
-            <mass value="8.34" />
-            <origin xyz="0 0 0.1" rpy="0 0 0" />
-            <inertia ixx="0.002386469" iyy="0.004827723" izz="0.003252219" ixy="0.0" ixz="0.0" iyz="0.0" />
-        </inertial>
-        <visual>
-            <geometry>
-                <mesh filename="package://my_amr/meshes/Base_final.stl"/>
+<?xml version="1.0"?>
+<robot name="amr" xmlns:xacro="http://ros.org/wiki/xacro" xmlns:xsi="http://www.w3.org/2001/XMLSchema-instance" xsi:noNamespaceSchemaLocation="http://wiki.ros.org/urdf/XML">
+    <!-- Include Gazebo Parameters -->
+    <xacro:include filename="$(find amr_description)/urdf/amr_gazebo.xacro" />
+    <!-- Include ros2_control Plugins -->
+    <xacro:include filename="$(find amr_description)/urdf/amr_ros2_control.xacro" />
+    <link name="base_footprint"/>
+    <link name="base_link">
+        <inertial>
+        <origin xyz="0 0 0.1" rpy="0 0 0" />
+        <mass value="8.34"/>
+        <inertia ixx="0.002386469" iyy="0.004827723" izz="0.003252219" ixy="0.0" ixz="0.0" iyz="0.0" />        </inertial>
+        <visual>
+        <origin xyz="0 0 0" rpy="0 0 0" />
+        <geometry>
+            <mesh filename="package://amr_description/meshes/Base_final.stl"/>
+        </geometry>
+        <material name="gray">
+            <color rgba=".7 .7 .7 1" />
+        </material>
+        </visual>
+        <collision>
+        <geometry>
+            <mesh filename="package://amr_description/meshes/Base_final.stl"/>
+        </geometry>
+        </collision>
+    </link>
+</link>
+<joint name="base_joint" type="fixed">
+<parent link="base_footprint"/>
+<child link="base"/>
+<origin rpy="0 0 0" xyz="0 0 0.093"/>
+</joint>
+    <!--
+    links for right front wheels
+    -->
+    <link name="shaft_right_front">
+        <inertial>
+        <mass value="0.06175"/>
+        <inertia ixx="0.000001112" iyy="0.000101416" izz="0.000101416" ixy="0.0" ixz="0.0" iyz="0.0"/>
+        <origin/>
+        </inertial>
+        <visual>
+            <geometry>
+                <mesh filename="package://amr_description/meshes/shaft_final.stl"/>
+            </geometry>
+            <material name="white">
+            <color rgba="1 1 1 1"/>
+            </material>
+        </visual>
+        <collision>
+            <geometry>
+                <mesh filename="package://amr_description/meshes/shaft_final.stl"/>
+            </geometry>
+            <contact_coefficients mu="0" kp="1000.0" kd="1.0"/>
+        </collision>
+        </link>
+    <link name="inner_right_front">
+        <inertial>
+        <mass value="0.94"/>
+        <inertia ixx="0.001752394" iyy="0.001233251" izz="0.001233251" ixy="0.0" ixz="0.0" iyz="0.0"/>
+        <origin/>
+        </inertial>
+        <visual>
+            <geometry>
+                <mesh filename="package://amr_description/meshes/inner_final.stl"/>
+            </geometry>
+            <material name="silver">
+            <color rgba="0.917647059 0.925490196 0.925490196 1"/>
+            </material>
+        </visual>
+        <collision>
+            <geometry>
+                <mesh filename="package://amr_description/meshes/inner_final.stl"/>
+            </geometry>
+            <contact_coefficients mu="0" kp="0.0" kd="0.0"/>
+        </collision>
+        </link>
+    <link name="outer_right_front">
+        <inertial>
+        <mass value="0.11614"/>
+        <inertia ixx="0.00036673" iyy="0.00036673" izz="0.000435441" ixy="0.0" ixz="0.0" iyz="0.0"/>
+        <origin/>
+        </inertial>
+        <visual>
+            <geometry>
+                <mesh filename="package://amr_description/meshes/outer_final.stl"/>
+            </geometry>
+            <material name="white">
+            <color rgba="0 0 0 1"/>
+            </material>
+        </visual>
+        <collision>
+            <geometry>
+                <mesh filename="package://amr_description/meshes/outer_final.stl"/>
+            </geometry>
+            <contact_coefficients mu="0" kp="0.0" kd="0.0"/>
+        </collision>
+        </link>
+    <!--
+    links for left front wheels
+    -->
+    <link name="shaft_left_front">
+        <inertial>
+        <mass value="0.06175"/>
+        <inertia ixx="0.000001112" iyy="0.000101416" izz="0.000101416" ixy="0.0" ixz="0.0" iyz="0.0"/>
+        <origin/>
+        </inertial>
+        <visual>
+            <geometry>
+                <mesh filename="package://amr_description/meshes/shaft_final.stl"/>
+            </geometry>
+            <material name="white">
+            <color rgba="1 1 1 1"/>
+            </material>
+        </visual>
+        <collision>
+            <geometry>
+                <mesh filename="package://amr_description/meshes/shaft_final.stl"/>
+            </geometry>
+            <contact_coefficients mu="0" kp="1000.0" kd="1.0"/>
+        </collision>
+        </link>
+    <link name="inner_left_front">
+        <inertial>
+        <mass value="0.94"/>
+        <inertia ixx="0.001752394" iyy="0.001233251" izz="0.001233251" ixy="0.0" ixz="0.0" iyz="0.0"/>
+        <origin/>
+        </inertial>
+        <visual>
+            <geometry>
+                <mesh filename="package://amr_description/meshes/inner_final.stl"/>
+            </geometry>
+            <material name="silver">
+            <color rgba="0.917647059 0.925490196 0.925490196 1"/>
+            </material>
+        </visual>
+        <collision>
+            <geometry>
+                <mesh filename="package://amr_description/meshes/inner_final.stl"/>
+            </geometry>
+            <contact_coefficients mu="0" kp="0.0" kd="0.0"/>
+        </collision>
+        </link>
+    <link name="outer_left_front">
+        <inertial>
+        <mass value="0.11614"/>
+        <inertia ixx="0.00036673" iyy="0.00036673" izz="0.000435441" ixy="0.0" ixz="0.0" iyz="0.0"/>
+        <origin/>
+        </inertial>
+        <visual>
+            <geometry>
+                <mesh filename="package://amr_description/meshes/outer_final.stl"/>
+            </geometry>
+            <material name="white">
+            <color rgba="0 0 0 1"/>
+            </material>
+        </visual>
+        <collision>
+            <geometry>
+                <mesh filename="package://amr_description/meshes/outer_final.stl"/>
+            </geometry>
+            <contact_coefficients mu="0" kp="0.0" kd="0.0"/>
+        </collision>
+        </link>
+    <!--
+    links for left back wheels
+    -->
+    <link name="shaft_left_back">
+        <inertial>
+        <mass value="0.06175"/>
+        <inertia ixx="0.000001112" iyy="0.000101416" izz="0.000101416" ixy="0.0" ixz="0.0" iyz="0.0"/>
+        <origin/>
+        </inertial>
+        <visual>
+            <geometry>
+                <mesh filename="package://amr_description/meshes/shaft_final.stl"/>
+            </geometry>
+            <material name="white">
+            <color rgba="1 1 1 1"/>
+            </material>
+        </visual>
+        <collision>
+            <geometry>
+                <mesh filename="package://amr_description/meshes/shaft_final.stl"/>
+            </geometry>
+            <contact_coefficients mu="0" kp="1000.0" kd="1.0"/>
+        </collision>
+        </link>
+    <link name="inner_left_back">
+        <inertial>
+        <mass value="0.94"/>
+        <inertia ixx="0.001752394" iyy="0.001233251" izz="0.001233251" ixy="0.0" ixz="0.0" iyz="0.0"/>
+        <origin/>
+        </inertial>
+        <visual>
+            <geometry>
+                <mesh filename="package://amr_description/meshes/inner_final.stl"/>
+            </geometry>
+            <material name="silver">
+            <color rgba="0.917647059 0.925490196 0.9254901961 1"/>
+            </material>
+        </visual>
+        <collision>
+            <geometry>
+                <mesh filename="package://amr_description/meshes/inner_final.stl"/>
+            </geometry>
+            <contact_coefficients mu="0" kp="0.0" kd="0.0"/>
+        </collision>
+        </link>
+    <link name="outer_left_back">
+        <inertial>
+        <mass value="0.11614"/>
+        <inertia ixx="0.00036673" iyy="0.00036673" izz="0.000435441" ixy="0.0" ixz="0.0" iyz="0.0"/>
+        <origin/>
+        </inertial>
+        <visual>
+            <geometry>
+                <mesh filename="package://amr_description/meshes/outer_final.stl"/>
+            </geometry>
+            <material name="white">
+            <color rgba="0 0 0 1"/>
+            </material>
+        </visual>
+        <collision>
+            <geometry>
+                <mesh filename="package://amr_description/meshes/outer_final.stl"/>
+            </geometry>
+            <contact_coefficients mu="0" kp="0.0" kd="0.0"/>
+        </collision>
+        </link>
+    <!--
+    links for right back wheels
+    -->
+    <link name="shaft_right_back">
+        <inertial>
+        <mass value="0.06175"/>
+        <inertia ixx="0.000001112" iyy="0.000101416" izz="0.000101416" ixy="0.0" ixz="0.0" iyz="0.0"/>
+        <origin/>
+        </inertial>
+        <visual>
+            <geometry>
+                <mesh filename="package://amr_description/meshes/shaft_final.stl"/>
+            </geometry>
+            <material name="white">
+            <color rgba="1 1 1 1"/>
+            </material>
+        </visual>
+        <collision>
+            <geometry>
+                <mesh filename="package://amr_description/meshes/shaft_final.stl"/>
+            </geometry>
+            <contact_coefficients mu="0" kp="1000.0" kd="1.0"/>
+        </collision>
+        </link>
+    <link name="inner_right_back">
+        <inertial>
+        <mass value="0.94"/>
+        <inertia ixx="0.001752394" iyy="0.001233251" izz="0.001233251" ixy="0.0" ixz="0.0" iyz="0.0"/>
+        <origin/>
+        </inertial>
+        <visual>
+            <geometry>
+                <mesh filename="package://amr_description/meshes/inner_final.stl"/>
+            </geometry>
+            <material name="silver">
+            <color rgba="0.917647059 0.925490196 0.925490196 1"/>
+            </material>
+        </visual>
+        <collision>
+            <geometry>
+                <mesh filename="package://amr_description/meshes/inner_final.stl"/>
+            </geometry>
+            <contact_coefficients mu="0" kp="0.0" kd="0.0"/>
+        </collision>
+        </link>
+    <link name="outer_right_back">
+        <inertial>
+        <mass value="0.11614"/>
+        <inertia ixx="0.00036673" iyy="0.00036673" izz="0.000435441" ixy="0.0" ixz="0.0" iyz="0.0"/>
+        <origin/>
+        </inertial>
+        <visual>
+            <geometry>
+                <mesh filename="package://amr_description/meshes/outer_final.stl"/>
+            </geometry>
+            <material name="white">
+            <color rgba="0 0 0 1"/>
+            </material>
+        </visual>
+        <collision>
+            <geometry>
+                <mesh filename="package://amr_description/meshes/outer_final.stl"/>
+            </geometry>
+            <contact_coefficients mu="0" kp="0.0" kd="0.0"/>
+        </collision>
+        </link>
+    <!--
+    link for top of the bot
+    -->
+    <link name="bot_top">
+        <inertial>
+        <mass value="8.47"/>
+        <inertia ixx="0.002307898" iyy="0.004479378" izz="0.002685416" ixy="0.0" ixz="0.0" iyz="0.0"/>
+        <origin/>
+        </inertial>
+        <visual>
+            <geometry>
+                <mesh filename="package://amr_description/meshes/top_final.stl"/>
+            </geometry>
+            <material name="gray">
+            <color rgba="0.7529 0.7529 0.7529 1"/>
+            </material>
+        </visual>
+        <collision>
+            <geometry>
+                <mesh filename="package://amr_description/meshes/top_final.stl"/>
+            </geometry>
+            <contact_coefficients mu="0" kp="0.0" kd="0.0"/>
+        </collision>
+        </link>
+    <!--
+    link for top of the bot plate
+    -->
+    <link name="bot_top_plate">
+        <inertial>
+        <mass value="2.54605"/>
+        <inertia ixx="0.000065178" iyy="0.000128019" izz="0.000065178" ixy="0.0" ixz="0.0" iyz="0.0"/>
+        <origin/>
+        </inertial>
+        <visual>
+            <geometry>
+                <mesh filename="package://amr_description/meshes/top_plate_final.stl"/>
             </geometry>
             <material name="gray">
@@ -17,322 +339,5 @@
         <collision>
             <geometry>
-                <mesh filename="package://my_amr/meshes/Base_final.stl"/>
-        </geometry>
-        <contact_coefficients mu="1" mu2="1" kp="1e+13.0" kd="1.0"/>
-        </collision>
-        </link>
-        <joint name="base_joint" type="fixed">
-        <parent link="base_footprint"/>
-        <child link="base"/>
-        <origin rpy="0 0 0" xyz="0 0 0.093"/>
-        </joint>
-    <!--
-    links for right front wheels
-    -->
-    <link name="shaft_right_front">
-        <inertial>
-        <mass value="0.06175"/>
-        <inertia ixx="0.000001112" iyy="0.000101416" izz="0.000101416" ixy="0.0" ixz="0.0" iyz="0.0"/>
-        <origin/>
-        </inertial>
-        <visual>
-            <geometry>
-                <mesh filename="package://my_amr/meshes/shaft_final.stl"/>
-            </geometry>
-            <material name="white">
-            <color rgba="1 1 1 1"/>
-            </material>
-        </visual>
-        <collision>
-            <geometry>
-                <mesh filename="package://my_amr/meshes/shaft_final.stl"/>
-            </geometry>
-            <contact_coefficients mu="0" kp="1000.0" kd="1.0"/>
-        </collision>
-        </link>
-    <link name="inner_right_front">
-        <inertial>
-        <mass value="0.94"/>
-        <inertia ixx="0.001752394" iyy="0.001233251" izz="0.001233251" ixy="0.0" ixz="0.0" iyz="0.0"/>
-        <origin/>
-        </inertial>
-        <visual>
-            <geometry>
-                <mesh filename="package://my_amr/meshes/inner_final.stl"/>
-            </geometry>
-            <material name="silver">
-            <color rgba="0.917647059 0.925490196 0.925490196 1"/>
-            </material>
-        </visual>
-        <collision>
-            <geometry>
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
Commit message: first pkg

File: src/amr_description/urdf/amr.urdf.xacro (robot description, xacro)
@@ -6,5 +6,5 @@
     <xacro:include filename="$(find amr_description)/urdf/amr_ros2_control.xacro" />
     <link name="base_footprint"/>
-    <link name="base_link">
+    <link name="base">
         <inertial>
         <origin xyz="0 0 0.1" rpy="0 0 0" />
@@ -26,10 +26,9 @@
         </collision>
     </link>
-</link>
-<joint name="base_joint" type="fixed">
-<parent link="base_footprint"/>
-<child link="base"/>
-<origin rpy="0 0 0" xyz="0 0 0.093"/>
-</joint>
+    <joint name="base_joint" type="fixed">
+    <parent link="base_footprint"/>
+    <child link="base"/>
+    <origin rpy="0 0 0" xyz="0 0 0.093"/>
+    </joint>
     <!--
     links for right front wheels

Commit message: optimize controller pkg

File: src/amr_description/urdf/amr.urdf.xacro (robot description, xacro)
@@ -498,5 +498,5 @@
     -->
         <joint name="kinect_camera_joint" type="fixed">
-        <origin xyz="0.23 0.0 0.07" rpy="0.0 0.0 3.14"/>
+        <origin xyz="0.23 0.0 0.07" rpy="0.0 0.0 0"/>
         <parent link="bot_top"/>
         <child link="kinect_camera"/>
