Commit message: fixing urdf file

File: install/amr_description/share/amr_description/urdf/amr.urdf.xacro (robot description, xacro)
@@ -10,5 +10,10 @@
         <origin xyz="0 0 0.1" rpy="0 0 0" />
         <mass value="8.34"/>
-        <inertia ixx="0.002386469" iyy="0.004827723" izz="0.003252219" ixy="0.0" ixz="0.0" iyz="0.0" />        </inertial>
+        <inertia ixx= "2386468.63e-7"
+        ixy = "-261456.79e-7"
+        iyy = "4827722.72e-7"
+        ixz= "76941.00e-7"
+        iyz = "57814.62e-7"
+        izz = "3252219.31e-7"/></inertial>
         <visual>
         <origin xyz="0 0 0" rpy="0 0 0" />
@@ -37,6 +42,11 @@
         <inertial>
         <mass value="0.06175"/>
-        <inertia ixx="0.000001112" iyy="0.000101416" izz="0.000101416" ixy="0.0" ixz="0.0" iyz="0.0"/>
-        <origin/>
+        <inertia
+        ixx="1111.52e-7"
+        iyy="101415.96e-7"
+        izz="101415.96e-7"
+        ixy="0.0"
+        ixz="0.0"
+        iyz="0.0"/>
         </inertial>
         <visual>
@@ -52,5 +62,4 @@
                 <mesh filename="package://amr_description/meshes/shaft_final.stl"/>
             </geometry>
-            <contact_coefficients mu="0" kp="1000.0" kd="1.0"/>
         </collision>
         </link>
@@ -58,6 +67,11 @@
         <inertial>
         <mass value="0.94"/>
-        <inertia ixx="0.001752394" iyy="0.001233251" izz="0.001233251" ixy="0.0" ixz="0.0" iyz="0.0"/>
-        <origin/>
+        <inertia
+        ixx="1752393.51e-7"
+        iyy="1233250.95e-7"
+        izz="1233250.94e-7"
+        ixy="-0.01e-7"
+        ixz="-0.05e-7"
+        iyz="0.1e-7"/>
         </inertial>
         <visual>
@@ -73,5 +87,4 @@
                 <mesh filename="package://amr_description/meshes/inner_final.stl"/>
             </geometry>
-            <contact_coefficients mu="0" kp="0.0" kd="0.0"/>
         </collision>
         </link>
@@ -79,33 +92,43 @@
         <inertial>
         <mass value="0.11614"/>
-        <inertia ixx="0.00036673" iyy="0.00036673" izz="0.000435441" ixy="0.0" ixz="0.0" iyz="0.0"/>
+        <inertia
+        ixx="366729.55e-7"
+        iyy="366729.55e-7"
+        izz="435440.86e-7"
+        ixy="0.0"
+        ixz="0.0"
+        iyz="0.0"/>
+        </inertial>
+        <visual>
+            <geometry>
+                <mesh filename="package://amr_description/meshes/outer_final.stl"/>
+            </geometry>
+            <material name="white">
+            <color rgba="0 0 0 1"/>
+            </material>
+        </visual>
+        <collision>
+            <geometry>
+                <mesh filename="package://amr_description/meshes/outer_final.stl"/>
+            </geometry>
+        </collision>
+        </link>
+    <!--
+    links for left front wheels
+    -->
+    <link name="shaft_left_front">
+        <inertial>
+        <mass value="0.06175"/>
+        <inertia
+        ixx="1111.52e-7"
+        iyy="101415.96e-7"
+        izz="101415.96e-7"
+        ixy="0.0"
+        ixz="0.0"
+        iyz="0.0"/>
         <origin/>
         </inertial>
         <visual>
             <geometry>
-                <mesh filename="package://amr_description/meshes/outer_final.stl"/>
-            </geometry>
-            <material name="white">
-            <color rgba="0 0 0 1"/>
-            </material>
-        </visual>
-        <collision>
-            <geometry>
-                <mesh filename="package://amr_description/meshes/outer_final.stl"/>
-            </geometry>
-            <contact_coefficients mu="0" kp="0.0" kd="0.0"/>
-        </collision>
-        </link>
-    <!--
-    links for left front wheels
-    -->
-    <link name="shaft_left_front">
-        <inertial>
-        <mass value="0.06175"/>
-        <inertia ixx="0.000001112" iyy="0.000101416" izz="0.000101416" ixy="0.0" ixz="0.0" iyz="0.0"/>
-        <origin/>
-        </inertial>
-        <visual>
-            <geometry>
                 <mesh filename="package://amr_description/meshes/shaft_final.stl"/>
             </geometry>
@@ -118,5 +141,4 @@
                 <mesh filename="package://amr_description/meshes/shaft_final.stl"/>
             </geometry>
-            <contact_coefficients mu="0" kp="1000.0" kd="1.0"/>
         </collision>
         </link>
@@ -124,6 +146,11 @@
         <inertial>
         <mass value="0.94"/>
-        <inertia ixx="0.001752394" iyy="0.001233251" izz="0.001233251" ixy="0.0" ixz="0.0" iyz="0.0"/>
-        <origin/>
+        <inertia
+        ixx="1752393.51e-7"
+        iyy="1233250.95e-7"
+        izz="1233250.94e-7"
+        ixy="-0.01e-7"
+        ixz="-0.05e-7"
+        iyz="0.1e-7"/>
         </inertial>
         <visual>
@@ -139,5 +166,4 @@
                 <mesh filename="package://amr_description/meshes/inner_final.stl"/>
             </geometry>
-            <contact_coefficients mu="0" kp="0.0" kd="0.0"/>
         </collision>
         </link>
@@ -145,33 +171,43 @@
         <inertial>
         <mass value="0.11614"/>
-        <inertia ixx="0.00036673" iyy="0.00036673" izz="0.000435441" ixy="0.0" ixz="0.0" iyz="0.0"/>
+        <inertia
+        ixx="366729.55e-7"
+        iyy="366729.55e-7"
+        izz="435440.86e-7"
+        ixy="0.0"
+        ixz="0.0"
+        iyz="0.0"/>
+        </inertial>
+        <visual>
+            <geometry>
+                <mesh filename="package://amr_description/meshes/outer_final.stl"/>
+            </geometry>
+            <material name="white">
+            <color rgba="0 0 0 1"/>
+            </material>
+        </visual>
+        <collision>
+            <geometry>
+                <mesh filename="package://amr_description/meshes/outer_final.stl"/>
+            </geometry>
+        </collision>
+        </link>
+    <!--
+    links for left back wheels
+    -->
+    <link name="shaft_left_back">
+        <inertial>
+        <mass value="0.06175"/>
+        <inertia
+        ixx="1111.52e-7"
+        iyy="101415.96e-7"
+        izz="101415.96e-7"
+        ixy="0.0"
+        ixz="0.0"
+        iyz="0.0"/>
         <origin/>
         </inertial>
         <visual>
             <geometry>
-                <mesh filename="package://amr_description/meshes/outer_final.stl"/>
-            </geometry>
-            <material name="white">
-            <color rgba="0 0 0 1"/>
-            </material>
-        </visual>
-        <collision>
-            <geometry>
-                <mesh filename="package://amr_description/meshes/outer_final.stl"/>
-            </geometry>
-            <contact_coefficients mu="0" kp="0.0" kd="0.0"/>
-        </collision>
-        </link>
-    <!--
-    links for left back wheels
-    -->
-    <link name="shaft_left_back">
-        <inertial>
-        <mass value="0.06175"/>
-        <inertia ixx="0.000001112" iyy="0.000101416" izz="0.000101416" ixy="0.0" ixz="0.0" iyz="0.0"/>
-        <origin/>
-        </inertial>
-        <visual>
-            <geometry>
                 <mesh filename="package://amr_description/meshes/shaft_final.stl"/>
             </geometry>
@@ -184,5 +220,4 @@
                 <mesh filename="package://amr_description/meshes/shaft_final.stl"/>
             </geometry>
-            <contact_coefficients mu="0" kp="1000.0" kd="1.0"/>
         </collision>
         </link>
@@ -190,6 +225,11 @@
         <inertial>
         <mass value="0.94"/>
-        <inertia ixx="0.001752394" iyy="0.001233251" izz="0.001233251" ixy="0.0" ixz="0.0" iyz="0.0"/>
-        <origin/>
+        <inertia
+        ixx="1752393.51e-7"
+        iyy="1233250.95e-7"
+        izz="1233250.94e-7"
+        ixy="-0.01e-7"
+        ixz="-0.05e-7"
+        iyz="0.1e-7"/>
         </inertial>
         <visual>
@@ -205,5 +245,4 @@
                 <mesh filename="package://amr_description/meshes/inner_final.stl"/>
             </geometry>
-            <contact_coefficients mu="0" kp="0.0" kd="0.0"/>
         </collision>
         </link>
@@ -211,33 +250,43 @@
         <inertial>
         <mass value="0.11614"/>
-        <inertia ixx="0.00036673" iyy="0.00036673" izz="0.000435441" ixy="0.0" ixz="0.0" iyz="0.0"/>
+        <inertia
+        ixx="366729.55e-7"
+        iyy="366729.55e-7"
+        izz="435440.86e-7"
+        ixy="0.0"
+        ixz="0.0"
+        iyz="0.0"/>
+        </inertial>
+        <visual>
+            <geometry>
+                <mesh filename="package://amr_description/meshes/outer_final.stl"/>
+            </geometry>
+            <material name="white">
+            <color rgba="0 0 0 1"/>
+            </material>
+        </visual>
+        <collision>
+            <geometry>
+                <mesh filename="package://amr_description/meshes/outer_final.stl"/>
+            </geometry>
+        </collision>
+        </link>
+    <!--
+    links for right back wheels
+    -->
+    <link name="shaft_right_back">
+        <inertial>
+        <mass value="0.06175"/>
+        <inertia
+        ixx="1111.52e-7"
+        iyy="101415.96e-7"
+        izz="101415.96e-7"
+        ixy="0.0"
+        ixz="0.0"
+        iyz="0.0"/>
         <origin/>
         </inertial>
         <visual>
             <geometry>
-                <mesh filename="package://amr_description/meshes/outer_final.stl"/>
-            </geometry>
-            <material name="white">
-            <color rgba="0 0 0 1"/>
-            </material>
-        </visual>
-        <collision>
-            <geometry>
-                <mesh filename="package://amr_description/meshes/outer_final.stl"/>
-            </geometry>
-            <contact_coefficients mu="0" kp="0.0" kd="0.0"/>
-        </collision>
-        </link>
-    <!--
-    links for right back wheels
-    -->
-    <link name="shaft_right_back">
-        <inertial>
-        <mass value="0.06175"/>
-        <inertia ixx="0.000001112" iyy="0.000101416" izz="0.000101416" ixy="0.0" ixz="0.0" iyz="0.0"/>
-        <origin/>
-        </inertial>
-        <visual>
-            <geometry>
                 <mesh filename="package://amr_description/meshes/shaft_final.stl"/>
             </geometry>
@@ -250,5 +299,4 @@
                 <mesh filename="package://amr_description/meshes/shaft_final.stl"/>
             </geometry>
-            <contact_coefficients mu="0" kp="1000.0" kd="1.0"/>
         </collision>
         </link>
@@ -256,6 +304,11 @@
         <inertial>
         <mass value="0.94"/>
-        <inertia ixx="0.001752394" iyy="0.001233251" izz="0.001233251" ixy="0.0" ixz="0.0" iyz="0.0"/>
-        <origin/>
+        <inertia
+        ixx="1752393.51e-7"
+        iyy="1233250.95e-7"
+        izz="1233250.94e-7"
+        ixy="-0.01e-7"
+        ixz="-0.05e-7"
+        iyz="0.1e-7"/>
         </inertial>
         <visual>
@@ -271,5 +324,4 @@
                 <mesh filename="package://amr_description/meshes/inner_final.stl"/>
             </geometry>
-            <contact_coefficients mu="0" kp="0.0" kd="0.0"/>
         </collision>
         </link>
@@ -277,6 +329,11 @@
         <inertial>
         <mass value="0.11614"/>
-        <inertia ixx="0.00036673" iyy="0.00036673" izz="0.000435441" ixy="0.0" ixz="0.0" iyz="0.0"/>
-        <origin/>
+        <inertia
+        ixx="366729.55e-7"
+        iyy="366729.55e-7"
+        izz="435440.86e-7"
+        ixy="0.0"
+        ixz="0.0"
+        iyz="0.0"/>
         </inertial>
         <visual>
@@ -292,5 +349,4 @@
                 <mesh filename="package://amr_description/meshes/outer_final.stl"/>
             </geometry>
-            <contact_coefficients mu="0" kp="0.0" kd="0.0"/>
         </collision>
         </link>
@@ -301,6 +357,11 @@
         <inertial>
         <mass value="8.47"/>
-        <inertia ixx="0.002307898" iyy="0.004479378" izz="0.002685416" ixy="0.0" ixz="0.0" iyz="0.0"/>
-        <origin/>
+        <inertia
+        ixx="2307897.72e-7"
+        iyy="4479377.88e-7"
+        izz="2685416.48e-7"
+        ixy="-25244.68e-7"
+        ixz="18060.35e-7"
+        iyz="-37339.81e-7"/>
         </inertial>
         <visual>
@@ -316,5 +377,4 @@
                 <mesh filename="package://amr_description/meshes/top_final.stl"/>
             </geometry>
-            <contact_coefficients mu="0" kp="0.0" kd="0.0"/>
         </collision>
         </link>
@@ -325,6 +385,11 @@
         <inertial>
         <mass value="2.54605"/>
-        <inertia ixx="0.000065178" iyy="0.000128019" izz="0.000065178" ixy="0.0" ixz="0.0" iyz="0.0"/>
-        <origin/>
+        <inertia
+        ixx="65177.65e-7"
+        iyy="128018.71e-7"
+        izz="65177.65e-7"
+        ixy="0.0"
+        ixz="0.0"
+        iyz="0.0"/>
         </inertial>
         <visual>
@@ -340,5 +405,4 @@
                 <mesh filename="package://amr_description/meshes/top_final.stl"/>
             </geometry>
-            <contact_coefficients mu="0" kp="0.0" kd="0.0"/>
         </collision>
         </link>
@@ -364,5 +428,4 @@
                 <mesh filename="package://amr_description/meshes/kinect.stl"/>
             </geometry>
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
File: install/amr_description/share/amr_description/urdf/amr_gazebo.xacro (robot description, xacro)
@@ -33,8 +33,8 @@
     <!-- Wheels -->
     <gazebo reference="shaft_right_back">
-    <mu1>1000000000000000.0</mu1>
-    <mu2>1000000000000000.0</mu2>
-    <kp>1000000000000.0</kp>
-    <kd>10.0</kd>
+    <mu1>0.0</mu1>
+    <mu2>0.0</mu2>
+    <kp>1000.0</kp>
+    <kd>1.0</kd>
     <minDepth>0.001</minDepth>
     <maxVel>0.1</maxVel>
@@ -42,8 +42,8 @@
     </gazebo>
     <gazebo reference="shaft_right_front">
-    <mu1>1000000000000000.0</mu1>
-    <mu2>1000000000000000.0</mu2>
-    <kp>1000000000000.0</kp>
-    <kd>10.0</kd>
+    <mu1>0.0</mu1>
+    <mu2>0.0</mu2>
+    <kp>1000.0</kp>
+    <kd>1.0</kd>
     <minDepth>0.001</minDepth>
     <maxVel>0.1</maxVel>
@@ -51,8 +51,8 @@
     </gazebo>
     <gazebo reference="shaft_left_back">
-    <mu1>1000000000000000.0</mu1>
-    <mu2>1000000000000000.0</mu2>
-    <kp>1000000000000.0</kp>
-    <kd>10.0</kd>
+    <mu1>0.0</mu1>
+    <mu2>0.0</mu2>
+    <kp>1000.0</kp>
+    <kd>1.0</kd>
     <minDepth>0.001</minDepth>
     <maxVel>0.1</maxVel>
@@ -60,12 +60,63 @@
     </gazebo>
     <gazebo reference="shaft_left_front">
-    <mu1>1000000000000000.0</mu1>
-    <mu2>1000000000000000.0</mu2>
-    <kp>1000000000000.0</kp>
-    <kd>10.0</kd>
+    <mu1>0.0</mu1>
+    <mu2>0.0</mu2>
+    <kp>1000.0</kp>
+    <kd>1.0</kd>
     <minDepth>0.001</minDepth>
     <maxVel>0.1</maxVel>
     <fdir1>1 0 0</fdir1>
     </gazebo>
+<gazebo reference="base">
+<material>Gazebo/Grey</material>
+</gazebo>
+<gazebo reference="bot_top">
+<material>Gazebo/Grey</material>
+</gazebo>
+<gazebo reference="shaft_right_front">
+<material>Gazebo/Grey</material>
+</gazebo>
+<gazebo reference="shaft_left_front">
+<material>Gazebo/Grey</material>
+</gazebo>
+<gazebo reference="shaft_right_back">
+<material>Gazebo/Grey</material>
+</gazebo>
+<gazebo reference="shaft_left_back">
+<material>Gazebo/Grey</material>
+</gazebo>
+<gazebo reference="inner_right_front">
+<material>Gazebo/White</material>
+</gazebo>
+<gazebo reference="inner_left_front">
+<material>Gazebo/White</material>
+</gazebo>
+<gazebo reference="inner_right_back">
+<material>Gazebo/White</material>
+</gazebo>
+<gazebo reference="inner_left_back">
+<material>Gazebo/White</material>
+</gazebo>
+<gazebo reference="outer_right_front">
+<material>Gazebo/Black</material>
+</gazebo>
+<gazebo reference="outer_left_front">
+<material>Gazebo/Black</material>
+</gazebo>
+<gazebo reference="outer_right_back">
+<material>Gazebo/Black</material>
+</gazebo>
+<gazebo reference="outer_left_back">
+<material>Gazebo/Black</material>
+</gazebo>
+<gazebo reference="bot_top_plate">
+<material>Gazebo/Grey</material>
+</gazebo>
+<gazebo reference="kinect_camera">
+<material>Gazebo/Black</material>
+</gazebo>
+<gazebo reference="lidar">
+<material>Gazebo/Black</material>
+</gazebo>
     <!-- ROS 2 Control -->
     <gazebo>
